File: CarLED_Atmega28/Car LEDs.kicad_pcb (KiCad board)
At the start: 2 copper layers, 108.6 x 47.9 mm, 73 parts, among them IC1 CP2102N-A02-GQFN24R, IC2 MCP4631-502E_ST, IC3 BLUETOOTH-SERIAL-HC-06, IC4 AP63356DV-7, IC5 AP7343DQ-33W5-7, J1 USB_B_Micro, J10 LED4_Pin9, J11 LED5_Pin10, J12 IO2, J13 Power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

Commit message: bumped kicad version
Other:
- net class Default removed
- board text added: "Pin ~10"
- board text added: "Pin ~3"
- board text added: "Pin ~5"
- board text added: "Pin ~6"
- board text added: "Pin ~9"
- board text added: "~D11 D12 D13"
- board text removed: "Pin ~~10"
- board text removed: "Pin ~~3"
- board text removed: "Pin ~~5"
- board text removed: "Pin ~~6"
- board text removed: "Pin ~~9"
- board text removed: "~~D11 D12 D13"
